Commit message: Migrated controller from tros2_control to gazebo ackermann-steering

File: src/car_model/urdf/controller.xacro (robot description, xacro)
@@ -1,40 +1,24 @@
 <?xml version="1.0"?>
 <robot xmlns:xacro="http://ros.org/wiki/xacro">
-	<ros2_control name="IgnitionSystem" type="system">
-		<hardware>
-			<plugin>ign_ros2_control/IgnitionSystem</plugin>
-		</hardware>
-		<joint name="front_left_wheel_steering_joint">
-			<command_interface name="position"/>
-			<state_interface name="position"/>
-		</joint>
-		<joint name="front_right_wheel_steering_joint">
-			<command_interface name="position"/>
-			<state_interface name="position"/>
-		</joint>
-		<joint name="rear_right_wheel_joint">
-			<command_interface name="velocity"/>
-			<state_interface name="position"/>
-			<state_interface name="velocity"/>
-		</joint>
-		<joint name="rear_left_wheel_joint">
-			<command_interface name="velocity"/>
-			<state_interface name="position"/>
-			<state_interface name="velocity"/>
-		</joint>
-		<!-- Need to add the other joints for JSB to publish-->
-		<joint name="front_left_wheel_joint">
-			<state_interface name="position"/>
-			<state_interface name="velocity"/>
-		</joint>
-		<joint name="front_right_wheel_joint">
-			<state_interface name="position"/>
-			<state_interface name="velocity"/>
-		</joint>
-	</ros2_control>
 	<gazebo>
-		<plugin filename="ign_ros2_control-system" name="ign_ros2_control::IgnitionROS2ControlPlugin">
-			<parameters>$(find car_model)/config/controller.yaml</parameters>
-			<controller_manager_name>controller_manager</controller_manager_name>
+		<plugin
+		filename="ignition-gazebo-ackermann-steering-system"
+		name="gz::sim::systems::AckermannSteering">
+			  <left_joint>front_left_wheel_joint</left_joint>
+			  <left_joint>rear_left_wheel_joint</left_joint>
+			  <right_joint>front_right_wheel_joint</right_joint>
+			  <right_joint>rear_right_wheel_joint</right_joint>
+			  <left_steering_joint>front_left_wheel_steering_joint</left_steering_joint>
+			  <right_steering_joint>front_right_wheel_steering_joint</right_steering_joint>
+			  <kingpin_width>0.07</kingpin_width>
+			  <steering_limit>0.4</steering_limit>
+			  <wheel_base>1.7</wheel_base>
+			  <wheel_separation>1.0</wheel_separation>
+			  <wheel_radius>0.30</wheel_radius>
+			  <min_velocity>-10.0</min_velocity>
+			  <max_velocity>10.0</max_velocity>
+			  <min_acceleration>-10</min_acceleration>
+			  <max_acceleration>10</max_acceleration>
+			  <topic>/cmd_vel</topic>
 		</plugin>
 	</gazebo>
