Commit message: Joint States publishing between Rviz andGazebo

File: src/car_model/urdf/gz_ackermann_demo.xacro.urdf (robot description, URDF)
Before this commit: robot vehicle_blue, 8 links, 7 joints
Joints:
- joint front_left_wheel_joint: origin (none) -> xyz=0 0.125029 -0.025 rpy=-1.5707 0 0
- joint front_left_wheel_steering_joint: origin (none) -> xyz=0.554283 0.5 0.02 rpy=0 0 0
- joint front_right_wheel_joint: origin (none) -> xyz=0 -0.125029 -0.025 rpy=-1.5707 0 0
- joint front_right_wheel_steering_joint: origin (none) -> xyz=0.554283 -0.5 0.02 rpy=0 0 0
- joint rear_left_wheel_joint: origin (none) -> xyz=-0.957138 0.625029 -0.025 rpy=-1.5707 0 0
- joint rear_right_wheel_joint: origin (none) -> xyz=-0.957138 -0.625029 -0.025 rpy=-1.5707 0 0
