Commit message: Updated Wheel size and Wheelbase parameters in URDF

File: src/car_model/urdf/gz_ackermann_controller.xacro (robot description, xacro)
@@ -14,5 +14,5 @@
 			<kingpin_width>1.0</kingpin_width>
 			<steering_limit>0.5</steering_limit>
-			<wheel_base>1.0</wheel_base>
+			<wheel_base>${wheel_base}</wheel_base>
 			<wheel_separation>1.25</wheel_separation>
 			<wheel_radius>0.3</wheel_radius>

File: src/car_model/urdf/gz_ackermann_demo.xacro.urdf (robot description, URDF)
Before this commit: robot vehicle_blue, 8 links, 7 joints
Links:
- link chassis_link: mass 1.14395 -> ${chassis_mass}; geometry collision box size=${chassis_length} ${chassis_width} ${chassis_height}; visual box size=${chassis_length} ${chassis_width} ${chassis_height}
- link front_left_wheel_link: mass 2 -> 5; geometry collision cylinder length=0.07 radius=0.3; visual cylinder length=0.07 radius=0.3
- link front_right_wheel_link: mass 2 -> 5; geometry collision cylinder length=0.07 radius=0.3; visual cylinder length=0.07 radius=0.3
- link rear_left_wheel_link: mass 2 -> 5; geometry collision cylinder length=0.07 radius=0.3; visual cylinder length=0.07 radius=0.3
- link rear_right_wheel_link: mass 2 -> 5; geometry collision cylinder length=0.07 radius=0.3; visual cylinder length=0.07 radius=0.3

Commit message: Ackermann Controller Working with Car Model

File: src/car_model/urdf/gz_ackermann_controller.xacro (robot description, xacro)
@@ -17,6 +17,6 @@
 			<wheel_separation>1.25</wheel_separation>
 			<wheel_radius>0.3</wheel_radius>
-			<min_velocity>-1</min_velocity>
-			<max_velocity>1</max_velocity>
+			<min_velocity>-5</min_velocity>
+			<max_velocity>5</max_velocity>
 			<min_acceleration>-3</min_acceleration>
 			<max_acceleration>3</max_acceleration>

File: src/car_model/urdf/gz_ackermann_demo.xacro.urdf (robot description, URDF)
Before this commit: robot vehicle_blue, 8 links, 7 joints
Joints:
- joint front_left_wheel_steering_joint: limit lower=-0.6 upper=0.6 effort=25 velocity=1.0 -> lower=-0.25 upper=0.25 effort=25 velocity=1.0; origin xyz=0.554283 0.5 0.02 rpy=0 0 0 -> xyz=${front_wheel_x} 0.5 0.02 rpy=0 0 0
- joint front_right_wheel_steering_joint: limit lower=-0.6 upper=0.6 effort=25 velocity=1.0 -> lower=-0.25 upper=0.25 effort=25 velocity=1.0; origin xyz=0.554283 -0.5 0.02 rpy=0 0 0 -> xyz=${front_wheel_x} -0.5 0.02 rpy=0 0 0
- joint rear_left_wheel_joint: origin xyz=-0.957138 0.625029 -0.025 rpy=-1.5707 0 0 -> xyz=${rear_wheel_x} 0.625029 -0.025 rpy=-1.5707 0 0
- joint rear_right_wheel_joint: origin xyz=-0.957138 -0.625029 -0.025 rpy=-1.5707 0 0 -> xyz=${rear_wheel_x} -0.625029 -0.025 rpy=-1.5707 0 0

Commit message: Updated Car Mesh

File: src/car_model/urdf/gz_ackermann_controller.xacro (robot description, xacro)
@@ -19,4 +19,5 @@
 			<min_velocity>-5</min_velocity>
 			<max_velocity>5</max_velocity>
+			<!-- Alter these acceleration values to create a more realistic speed change -->
 			<min_acceleration>-3</min_acceleration>
 			<max_acceleration>3</max_acceleration>

File: src/car_model/urdf/gz_ackermann_demo.xacro.urdf (robot description, URDF)
Before this commit: robot vehicle_blue, 8 links, 7 joints
Links:
- link chassis_link: geometry collision box size=${chassis_length} ${chassis_width} ${chassis_height}; visual mesh filename=package://car_model/meshes/chassis.stl scale=0.002 0.001 0.001
