Commit message: Improved car's visuals

File: src/car_model/urdf/AV_car.xacro.urdf (robot description, URDF)
Before this commit: robot FYP_car, 2 links, 1 joints
Links:
- removed link world_link
- added link chassis_link; collision box size=${chassis_length} ${chassis_width_bottom} ${chassis_height}; visual mesh filename=package://car_model/meshes/chassis.stl scale=0.002 0.001 0.001
- link base_link: geometry 
Joints:
- joint base_joint: child base_link -> chassis_link; parent world_link -> base_link

File: src/car_model/urdf/ackermann_joints.xacro (robot description, xacro)
@@ -7,5 +7,5 @@
 		<joint name="${suffix}_wheel_steering_joint" type="revolute">
 			<xacro:insert_block name="origin"/>
-			<parent link="base_link" />
+			<parent link="chassis_link" />
 			<child link="${suffix}_wheel_steering_link" />
 			<axis xyz="0 0 1" />

File: src/car_model/urdf/wheel.xacro (robot description, xacro)
@@ -17,6 +17,6 @@
 				</geometry>
 				<origin xyz="0.0 0.0 0.0" rpy="0 0 0" />
-				<material name="blue">
-					<color rgba="0 0.5 0.25 0.5"/>
+				<material name="black">
+					<color rgba="0 0 0 0.5"/>
 				</material>
 			</visual>

Commit message: STL model loaded by both Gazebo and Rviz
Had to add the path ${package}/src/mesh to .bashrc
JSP removed

File: src/car_model/urdf/AV_car.xacro.urdf (robot description, URDF)
Before this commit: robot FYP_car, 2 links, 1 joints
Links:
- link chassis_link: mass None -> 100

Commit message: Controls Implemented, BUG: Car not doing translation, just steering front wheels

File: src/car_model/urdf/AV_car.xacro.urdf (robot description, URDF)
Before this commit: robot FYP_car, 2 links, 1 joints
Links:
- link chassis_link: geometry collision box size=${chassis_length} ${chassis_width_bottom} ${chassis_height}; visual box size=${chassis_length} ${chassis_width_bottom} ${chassis_height}
Joints:
- removed joint base_joint
- added joint chassis_joint: type fixed, parent base_link, child chassis_link, origin xyz=0 0 ${ground_clearance}

File: src/car_model/urdf/ackermann_joints.xacro (robot description, xacro)
@@ -11,5 +11,5 @@
 			<axis xyz="0 0 1" />
 			<!-- change effort after you we know the value of torquw -->
-			<limit lower="${radians(-14.3)}" upper="${radians(14.3)}" velocity="5.56" effort="100" />
+			<limit lower="${radians(-14.3)}" upper="${radians(14.3)}" velocity="30" effort="1000.0" />
 		</joint>
 		<link name="${suffix}_wheel_steering_link">

File: src/car_model/urdf/wheel.xacro (robot description, xacro)
@@ -6,8 +6,9 @@
 	<xacro:macro name="wheel" params="suffix direction parent *origin">
 		<joint name="${suffix}_${direction}_wheel_joint" type="continuous">
+			<axis xyz="0 0 1"/>
 			<xacro:insert_block name="origin"/>
 			<parent link="${parent}"/>
 			<child link="${suffix}_${direction}_wheel_link"/>
-			<axis xyz="0 0 1"/>
+			<dynamics damping="0.2" />
 		</joint>
 		<link name="${suffix}_${direction}_wheel_link">
@@ -30,6 +31,5 @@
 			<inertial>
 				<mass value="5.0"/>
-				<origin xyz="0.0 0.0 0.0" rpy="0 0 0" />
-				<inertia ixx="0.452" ixy="0.0" ixz="0.0" iyy="0.452" iyz="0.0" izz="0.9" />
+				<inertia ixx="${(3*radius*radius + thickness*thickness)*5/12}" ixy="0.0" ixz="0.0" iyy="${(3*radius*radius + thickness*thickness)*5/12}" iyz="0.0" izz="${5*radius*radius/2}" />
 			</inertial>
 		</link>

Commit message: Lidar sensor integrated in gazebo + File names changed

File: src/car_model/urdf/AV_car.xacro.urdf (robot description, URDF)
Before this commit: robot vehicle_blue, 8 links, 7 joints
Links:
- added link lidar_link, mass 0.425; collision cylinder length=0.0735 radius=0.04; visual cylinder length=0.0735 radius=0.04
Joints:
- added joint lidar_joint: type continuous, parent chassis_link, child lidar_link, origin xyz=-0.05 0 1.305, axis 0 0 1

File: src/car_model/urdf/gz_plugins.xacro (robot description, xacro)
@@ -35,5 +35,55 @@
 			<joint_name>rear_left_wheel_joint</joint_name>
 			<joint_name>rear_right_wheel_joint</joint_name>
+			<joint_name>lidar_joint</joint_name>
 		</plugin>
 	</gazebo>
+	<!--
+	<gazebo>
+	  <plugin
+        filename="ignition-gazebo-apply-joint-force-system"
+        name="gz::sim::systems::ApplyJointForce">
+        <joint_name>lidar_joint</joint_name>
+      </plugin>
+	</gazebo>
+	-->
+	<gazebo>
+		<plugin
+		  filename="libignition-gazebo-sensors-system.so"
+		  name="ignition::gazebo::systems::Sensors">
+			  <render_engine>ogre2</render_engine>
+		</plugin>
+	</gazebo>
+	<gazebo reference="lidar_link">
+		<sensor name="lidar_link" type="gpu_lidar">
+		  <pose relative_to='lidar_link'>0 0 0 0 0 0</pose>
+		  <topic>/lidar</topic>
+		  <update_rate>10</update_rate>
+		  <ray>
+			<scan>
+			  <horizontal>
+				  <samples>15</samples>
+				  <resolution>1</resolution>
+				  <min_angle>-3.141592654</min_angle>
+				  <max_angle>3.141592654</max_angle>
+			  </horizontal>
+			  <vertical>
+				  <samples>16</samples>
+				  <resolution>1</resolution>
+				  <min_angle>-0.2897256658</min_angle>
+				  <max_angle>0.2897256658</max_angle>
+			  </vertical>
+			</scan>
+			<range>
+				<min>0.2</min>
+				<max>15.0</max>
+				<resolution>0.001</resolution>
+			</range>
+		  </ray>
+		  <always_on>1</always_on>
+		  <visualize>true</visualize>
+		  <frame_id>lidar_link</frame_id>
+		  <gz_frame_id>lidar_link</gz_frame_id>
+		  <ign_frame_id>lidar_link</ign_frame_id>
+		</sensor>
+	</gazebo>
 </robot>

Commit message: Added IMU to simulation

File: src/car_model/urdf/AV_car.xacro.urdf (robot description, URDF)
Before this commit: robot vehicle_blue, 9 links, 8 joints
Links:
- added link imu_link, mass 0.425
Joints:
- added joint imu_joint: type continuous, parent chassis_link, child imu_link, origin xyz=-0.05 0 1.305, axis 0 0 1

File: src/car_model/urdf/gz_plugins.xacro (robot description, xacro)
@@ -36,4 +36,5 @@
 			<joint_name>rear_right_wheel_joint</joint_name>
 			<joint_name>lidar_joint</joint_name>
+			<joint_name>imu_joint</joint_name>
 		</plugin>
 	</gazebo>
@@ -87,3 +88,17 @@
 		</sensor>
 	</gazebo>
+	<!-- IMU -->
+	<gazebo>
+		<plugin filename="libignition-gazebo-imu-system.so"
+        name="ignition::gazebo::systems::Imu">
+		</plugin>
+	</gazebo>
+	<gazebo reference="imu_link">
+		<sensor name="imu_link" type="imu">
+			<always_on>1</always_on>
+			<update_rate>1</update_rate>
+			<visualize>true</visualize>
+			<topic>imu</topic>
+		</sensor>
+	</gazebo>
 </robot>

Commit message: Module up to date

File: src/car_model/urdf/AV_car.xacro.urdf (robot description, URDF)
Before this commit: robot vehicle_blue, 10 links, 9 joints
Joints:
- joint imu_joint: type continuous -> fixed
- joint lidar_joint: axis 0 0 1 -> (none); origin xyz=-0.05 0 1.305 -> xyz=-0.05 0 1.38; type continuous -> fixed

File: src/car_model/urdf/gz_plugins.xacro (robot description, xacro)
@@ -35,6 +35,4 @@
 			<joint_name>rear_left_wheel_joint</joint_name>
 			<joint_name>rear_right_wheel_joint</joint_name>
-			<joint_name>lidar_joint</joint_name>
-			<joint_name>imu_joint</joint_name>
 		</plugin>
 	</gazebo>
@@ -63,5 +61,5 @@
 			<scan>
 			  <horizontal>
-				  <samples>512</samples>
+				  <samples>1024</samples>
 				  <resolution>1</resolution>
 				  <min_angle>-3.141592654</min_angle>
@@ -69,5 +67,5 @@
 			  </horizontal>
 			  <vertical>
-				  <samples>16</samples>
+				  <samples>64</samples>
 				  <resolution>1</resolution>
 				  <min_angle>-0.2897256658</min_angle>
